File: hardware/sfp-receiver/sfp-receiver.kicad_pcb (KiCad board)
At the start: 2 copper layers, 100 x 50 mm, 32 parts, among them J1 SFP, J2 CLK1, J3 CLK2, J6 Jack-DC, U1 SN65MLVD200AD, U2 LT1117-3.3, U3 74LVC1GU04DRL, U4 74LVC2G17

Commit message: feat(LMPT-contraption): revision A
Routing:
- net GND: track 38.3 -> 54.7 mm
Changed lines of the file:
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@@
-	)
-	(segment
-		(start 177.65 76.825)
-		(end 177.65 77.7)
-		(width 0.3)
-		(layer "F.Cu")
-		(net 1)
-	)
-	(segment
-		(start 177.4625 74)
-		(end 178.376 74)
-		(width 0.3)
-		(layer "F.Cu")
-		(net 1)
 	)
 	(segment
@@
 	)
 	(segment
+		(start 160.6625 71.45)
+		(end 178.15 71.45)
+		(width 0.3)
+		(layer "F.Cu")
+		(net 1)
+	)
+	(segment
 		(start 142.1 67.45)
 		(end 142.1 68.85)
@@
 	)
 	(segment
-		(start 178.376 74)
-		(end 178.376 76.099)
-		(width 0.3)
-		(layer "F.Cu")
-		(net 1)
-	)
-	(segment
-		(start 178.376 76.099)
-		(end 177.65 76.825)
+		(start 178.15 71.45)
+		(end 178.7 72)
+		(width 0.3)
+		(layer "F.Cu")
+		(net 1)
+	)
+	(segment
+		(start 178.3125 74)
+		(end 177.4625 74)
+		(width 0.3)
+		(layer "F.Cu")
+		(net 1)
+	)
+	(segment
+		(start 178.7 72)
+		(end 178.7 73.6125)
 		(width 0.3)
 		(layer "F.Cu")
@@
 		(start 111.8 58.45)
 		(end 111.8 56)
+		(width 0.3)
+		(layer "F.Cu")
+		(net 1)
+	)
+	(segment
+		(start 178.7 73.6125)
+		(end 178.3125 74)
 		(width 0.3)
 		(layer "F.Cu")
@@
 	)
 	(segment
+		(start 179.7375 74)
+		(end 179.021021 74)
+		(width 0.3)
+		(layer "F.Cu")
+		(net 20)
+	)
+	(segment
 		(start 145.2 61.65)
 		(end 150.65 61.65)
@@
 	)
 	(segment
+		(start 179.55 76.75)
+		(end 179.55 77.7)
+		(width 0.3)
+		(layer "F.Cu")
+		(net 20)
+	)
+	(segment
 		(start 140 87.1)
 		(end 140 84.6)
@@
 	)
 	(segment
-		(start 178.824 74)
-		(end 178.824 76.024)
-		(width 0.3)
-		(layer "F.Cu")
-		(net 20)
-	)
-	(segment
 		(start 144.4 58.2)
 		(end 145.2 59)
@@
 	)
 	(segment
-		(start 178.824 76.024)
-		(end 179.55 76.75)
-		(width 0.3)
-		(layer "F.Cu")
-		(net 20)
-	)
-	(segment
-		(start 179.7375 74)
-		(end 178.824 74)
-		(width 0.3)
-		(layer "F.Cu")
-		(net 20)
-	)
-	(segment
 		(start 150.65 74)
 		(end 153.049938 74)
@@
 	)
 	(segment
+		(start 178.52002 75.72002)
+		(end 179.55 76.75)
+		(width 0.3)
+		(layer "F.Cu")
+		(net 20)
+	)
+	(segment
+		(start 178.52002 74.501)
+		(end 178.52002 75.72002)
+		(width 0.3)
+		(layer "F.Cu")
+		(net 20)
+	)
+	(segment
 		(start 130.3125 55.7125)
 		(end 130.625 56.025)
@@
 	)
 	(segment
-		(start 179.55 76.75)
-		(end 179.55 77.7)
-		(width 0.3)
-		(layer "F.Cu")
+		(start 179.021021 74)
+		(end 178.52002 74.501)
+		(width 0.3)
+		(layer "F.Cu")
