File: hardware/sfp-receiver/sfp-receiver.kicad_sch (KiCad schematic)
At the start: 32 parts, among them J1 SFP, J2 CLK1, J3 CLK2, J6 Jack-DC, U1 SN65MLVD200AD, U2 LT1117-3.3, U3 74LVC1GU04DRL, U4 74LVC2G17

Commit message: feat(LMPT-contraption): revision A
Parts:
- removed R4: 100K, Resistor_SMD:R_0805_2012Metric, symbol Device:R
- removed TP2: GND, TestPoint:TestPoint_Pad_1.5x1.5mm, symbol Connector:TestPoint
