File: hardware/lmpt-contraption/lmpt-contraption.kicad_pcb (KiCad board)
At the start: 2 copper layers, 62 x 62 mm, 22 parts, among them IC1 SN74LVC541APW, J1 CLK_IN, J2 CLK_A, J3 CLK_B, J4 1PPS Out Conn, J5 RPi Out Conn, U1 LT1117-3.3, U2 74LVC2G17

Commit message: feat(LMPT-contraption): revision B
Parts:
- removed C4: 0.1uF 6.3V, Capacitor_SMD:C_0805_2012Metric
- removed IC1: SN74LVC541APW, Package_SO:TSSOP-20_4.4x6.5mm_P0.65mm
- removed J4: 1PPS Out Conn, Connector_PinHeader_2.54mm:PinHeader_2x04_P2.54mm_Vertical_SMD
- removed TP5: GND, TestPoint:TestPoint_Pad_2.0x2.0mm
- added C5: 0.1uF 6.3V, Capacitor_SMD:C_0805_2012Metric, F.Cu at (133.8, 109.3)
- added J6: CLK_D, Connector_Coaxial:U.FL_Molex_MCRF_73412-0110_Vertical, F.Cu at (125.2, 120.3)
- added J7: CLK_C, Connector_Coaxial:U.FL_Molex_MCRF_73412-0110_Vertical, F.Cu at (109.8, 120.3)
- added J9: PPS_OUT, Connector_PinHeader_2.54mm:PinHeader_2x03_P2.54mm_Vertical_SMD, F.Cu at (149.5, 98.8)
- added TP3: GNSS_PPS, TestPoint:TestPoint_Pad_D2.0mm, F.Cu at (132.2, 114.1)
- added U3: CDCV304, Package_SO:TSSOP-8_4.4x3mm_P0.65mm, F.Cu at (118.5, 106.2)
- J2, J3: footprint Connector_Coaxial:U.FL_Molex_MCRF_73412-0110_Vertical -> Connector_Coaxial:SMA_Molex_73251-1153_EdgeMount_Horizontal
- J5: value RPi Out Conn -> RPI_CONN
- TP4: value 1PPS -> GNSS_GND; footprint TestPoint:TestPoint_Pad_D2.0mm -> TestPoint:TestPoint_Pad_2.0x2.0mm
- U2: value 74LVC2G17 -> CDCV304; footprint Package_TO_SOT_SMD:SOT-23-6 -> Package_SO:TSSOP-8_4.4x3mm_P0.65mm
- moved J3 46.5 mm to (100.0, 113.8), turned to 0 degrees
- moved J1 46.1 mm to (117.5, 120.3), turned to 180 degrees
- moved J2 38.3 mm to (100.1, 98.0), turned to 0 degrees
- moved U2 22.9 mm to (137.0, 111.2), turned to 90 degrees
- moved C3 21.9 mm to (116.6, 102.8), turned to 180 degrees
- moved C2 16.9 mm to (117.5, 91.5), turned to 90 degrees
- moved TP4 16.5 mm to (132.2, 118.2), turned to 180 degrees
- moved C1 15.8 mm to (126.2, 86.5), turned to 180 degrees
- moved TP1 14.3 mm to (131.3, 90.2), turned to 180 degrees
- moved TP2 11.6 mm to (131.3, 94.8), turned to 180 degrees
- moved U1 4.77 mm to (124.0, 92.5), turned to 180 degrees
Connections:
- J1 pad 1: /CLK_IN -> Net-(J1-In)
- J5 pad 4: Net-(IC1-Y5) -> Net-(J5-Pin_4)
- TP4 pad 1: Net-(IC1-A1) -> GND
- U2 pad 1: /CLK_IN -> Net-(U2-CLKIN)
- U2 pad 2: GND -> +3V3
- U2 pad 3: /CLK_IN -> Net-(J5-Pin_4)
- U2 pad 4: Net-(J3-In) -> GND
- U2 pad 5: +3V3 -> Net-(J9-Pin_5)
- U2 pad 6: Net-(J2-In) -> +3V3
Routing:
- net Net-(IC1-A1): track 79.2 -> 0.00 mm
- net GND: track 28.2 -> 0.00 mm
- net Net-(IC1-Y5): track 22.4 -> 0.00 mm
- net Net-(IC1-Y2): track 22.4 -> 0.00 mm
- net Net-(IC1-Y1): track 22.3 -> 0.00 mm
- net Net-(IC1-Y3): track 22.3 -> 0.00 mm
- net Net-(IC1-Y4): track 22.2 -> 0.00 mm
- net Net-(J5-Pin_4): track 0.00 -> 20.0 mm
- net Net-(J9-Pin_1): track 0.00 -> 19.9 mm
- net Net-(J9-Pin_3): track 0.00 -> 19.9 mm
- net Net-(J9-Pin_5): track 0.00 -> 19.8 mm
- net Net-(J6-In): track 0.00 -> 16.1 mm
- net Net-(J3-In): track 5.11 -> 20.3 mm
- net Net-(J2-In): track 5.11 -> 20.3 mm
- net Net-(J7-In): track 0.00 -> 14.0 mm
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
Commit message: feat(LMTP-contraption): Revision E
Parts:
- removed C5: 0.1uF 6.3V, Capacitor_SMD:C_0805_2012Metric
- removed J5: RPI_CONN, Connector_PinHeader_2.54mm:PinHeader_1x04_P2.54mm_Horizontal
- removed J6: CLK_D, Connector_Coaxial:U.FL_Molex_MCRF_73412-0110_Vertical
- removed J7: CLK_C, Connector_Coaxial:U.FL_Molex_MCRF_73412-0110_Vertical
- removed J9: PPS_OUT, Connector_PinHeader_2.54mm:PinHeader_2x03_P2.54mm_Vertical_SMD
- removed TP4: GNSS_GND, TestPoint:TestPoint_Pad_2.0x2.0mm
- removed U3: CDCV304, Package_SO:TSSOP-8_4.4x3mm_P0.65mm
- added C4: 0.1uF 6.3V, Capacitor_SMD:C_0805_2012Metric, F.Cu at (115.8, 105.0)
- added H5: B.Cu Via, BKSP:Hole_Via_0.8mm, F.Cu at (153.0, 103.0)
- added H6: B.Cu Via, BKSP:Hole_Via_0.8mm, F.Cu at (109.5, 102.5)
- added IC1: SN74LVC541APW, Package_SO:TSSOP-20_4.4x6.5mm_P0.65mm, F.Cu at (139.0, 120.0)
- added J4: Conn_02x04_Odd_Even, Connector_PinSocket_2.54mm:PinSocket_2x04_P2.54mm_Vertical_SMD, F.Cu at (123.9, 118.5)
- added TP5: GNSS_TXD, BKSP:BKSP_TestPoint_Pad_5mm_2.5mm, F.Cu at (153.0, 108.7)
- J1: footprint Connector_Coaxial:U.FL_Molex_MCRF_73412-0110_Vertical -> BKSP:Connector_RF_UFL_SMT160
- TP1: footprint TestPoint:TestPoint_Pad_D2.0mm -> BKSP:BKSP_TestPoint_Pad_5mm_2.5mm
- TP2: footprint TestPoint:TestPoint_Pad_2.0x2.0mm -> BKSP:BKSP_TestPoint_Pad_5mm_2.5mm
- TP3: value GNSS_PPS -> GNSS_GND; footprint TestPoint:TestPoint_Pad_D2.0mm -> BKSP:BKSP_TestPoint_Pad_5mm_2.5mm
- TP6: footprint TestPoint:TestPoint_Pad_1.5x1.5mm -> BKSP:BKSP_TestPoint_Pad_5mm_2.5mm
- TP7: value GNSS_TXD -> GNSS_PPS; footprint TestPoint:TestPoint_Pad_D1.5mm -> BKSP:BKSP_TestPoint_Pad_5mm_2.5mm
- U2: value CDCV304 -> 74LVC2G17; footprint Package_SO:TSSOP-8_4.4x3mm_P0.65mm -> Package_TO_SOT_SMD:SOT-23-6
- moved C3 25.3 mm to (139.2, 114.2), turned to 0 degrees
- moved U2 25.3 mm to (112.2, 106.0), turned to 0 degrees
- moved TP2 21.9 mm to (153.0, 98.0)
- moved TP1 21.8 mm to (153.0, 92.7)
- moved TP3 21.4 mm to (153.0, 119.4), turned to 0 degrees
- moved J1 20.9 mm to (102.2, 106.0), turned to 90 degrees
- moved C2 20.2 mm to (137.7, 94.0)
- moved U1 20.2 mm to (144.2, 95.0)
- moved C1 20.2 mm to (146.3, 89.0)
- moved TP6 8.14 mm to (153.0, 124.8)
- moved TP7 6.48 mm to (153.0, 114.0)
- moved J3 4.76 mm to (99.7, 118.5)
- moved J2 4.51 mm to (99.7, 93.5)
Connections:
- C3 pad 1: +3V3 -> GND
- C3 pad 2: GND -> +3V3
- TP3 pad 1: Net-(U2-CLKIN) -> GND
- TP6 pad 1: Net-(J5-Pin_3) -> /GNSS_RXD
- TP7 pad 1: Net-(J5-Pin_2) -> /GNSS_PPS
- U2 pad 1: Net-(U2-CLKIN) -> Net-(J1-In)
- U2 pad 2: +3V3 -> GND
- U2 pad 3: Net-(J5-Pin_4) -> Net-(J1-In)
- U2 pad 4: GND -> Net-(J3-In)
- U2 pad 5: Net-(J9-Pin_5) -> +3V3
- U2 pad 6: +3V3 -> Net-(J2-In)
Routing:
- net GND: track 0.00 -> 42.0 mm, vias 4 -> 0
- net /GNSS_RXD: track 0.00 -> 33.7 mm
- net /TXD_B: track 0.00 -> 22.2 mm
- net /GNSS_TXD: track 0.00 -> 20.0 mm
- net Net-(J5-Pin_4): track 20.0 -> 0.00 mm
- net Net-(J9-Pin_1): track 19.9 -> 0.00 mm
- net Net-(J9-Pin_3): track 19.9 -> 0.00 mm
- net Net-(J9-Pin_5): track 19.8 -> 0.00 mm
- net /TXD_A: track 0.00 -> 19.2 mm
- net Net-(J6-In): track 16.1 -> 0.00 mm
- net /GNSS_PPS: track 0.00 -> 14.1 mm
- net Net-(J7-In): track 14.0 -> 0.00 mm
- net /PPS_B: track 0.00 -> 9.96 mm
- net /PPS_A: track 0.00 -> 9.96 mm
- net +3V3: track 58.4 -> 68.1 mm
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